File: Hardware - MultiStar, 5 points/Qwiic_MultiStar.brd (EAGLE design)
At the start: 64.8 x 59.7 mm, 23 parts, among them J1 QWIIC_RIGHT_ANGLE, J2 QWIIC_RIGHT_ANGLE, J3 QWIIC_RIGHT_ANGLE, J4 QWIIC_RIGHT_ANGLE, J5 QWIIC_RIGHT_ANGLE

Commit message: re-route MultiPort in daisy chain configuration
Parts:
- moved LOGO3 0.64 mm to (32.4, 20.3)
Changed lines of the file:
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@@
 <?xml version="1.0" encoding="utf-8"?>
 <!DOCTYPE eagle SYSTEM "eagle.dtd">
-<eagle version="9.6.2">
+<eagle version="9.5.2">
 <drawing>
 <settings>
@@
 <element name="LOGO1" library="SparkFun-Aesthetics" package="QWIIC_5MM" value="QWIIC_LOGO_5MM" x="57.15" y="38.1" smashed="yes" rot="MR0"/>
 <element name="LOGO2" library="SparkFun-Aesthetics" package="QWIIC_5MM" value="QWIIC_LOGO_5MM" x="57.15" y="38.1" smashed="yes"/>
-<element name="LOGO3" library="SparkFun-Aesthetics" package="OSHW-LOGO-S" value="OSHW-LOGOS" x="33.02" y="20.32" smashed="yes" rot="MR0"/>
+<element name="LOGO3" library="SparkFun-Aesthetics" package="OSHW-LOGO-S" value="OSHW-LOGOS" x="32.385" y="20.32" smashed="yes" rot="MR0"/>
 <element name="LOGO4" library="SparkFun-Aesthetics" package="SFE_LOGO_NAME_.2" value="SFE_LOGO_NAME.2_INCH" x="33.02" y="29.21" smashed="yes" rot="MR0"/>
 <element name="J5" library="SparkFun-Connectors" package="JST04_1MM_RA" value="QWIIC_RIGHT_ANGLE" x="33.401" y="45.72" smashed="yes" rot="R114.8">

Commit message: Update silkscreen
Parts:
- added U$1: (no value), output:OSHW_NOT_OSHA0
- moved LOGO3 1.27 mm to (32.4, 21.6)
- moved U$5 0.89 mm to (37.6, 26.7)
- moved U$3 0.89 mm to (27.2, 26.7)
Changed lines of the file:
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@@
 <?xml version="1.0" encoding="utf-8"?>
 <!DOCTYPE eagle SYSTEM "eagle.dtd">
-<eagle version="9.5.2">
+<eagle version="9.6.2">
 <drawing>
 <settings>
@@
 <element name="LOGO1" library="SparkFun-Aesthetics" package="QWIIC_5MM" value="QWIIC_LOGO_5MM" x="57.15" y="38.1" smashed="yes" rot="MR0"/>
 <element name="LOGO2" library="SparkFun-Aesthetics" package="QWIIC_5MM" value="QWIIC_LOGO_5MM" x="57.15" y="38.1" smashed="yes"/>
-<element name="LOGO3" library="SparkFun-Aesthetics" package="OSHW-LOGO-S" value="OSHW-LOGOS" x="32.385" y="20.32" smashed="yes" rot="MR0"/>
+<element name="LOGO3" library="SparkFun-Aesthetics" package="OSHW-LOGO-S" value="OSHW-LOGOS" x="32.385" y="21.59" smashed="yes" rot="MR0"/>
 <element name="LOGO4" library="SparkFun-Aesthetics" package="SFE_LOGO_NAME_.2" value="SFE_LOGO_NAME.2_INCH" x="33.02" y="29.21" smashed="yes" rot="MR0"/>
 <element name="J5" library="SparkFun-Connectors" package="JST04_1MM_RA" value="QWIIC_RIGHT_ANGLE" x="33.401" y="45.72" smashed="yes" rot="R114.8">
@@
 </element>
 <element name="U$2" library="SparkFun-Aesthetics" package="SFE_LOGO_FLAME_.2" value="" x="33.02" y="21.59" smashed="yes"/>
-<element name="U$3" library="output" package="MULTISTAR0" value="" x="28.067" y="26.67" smashed="yes"/>
-<element name="U$5" library="output" package="MULTISTAR0" value="" x="38.481" y="26.67" smashed="yes" rot="MR0"/>
+<element name="U$3" library="output" package="MULTISTAR0" value="" x="27.178" y="26.67" smashed="yes"/>
+<element name="U$5" library="output" package="MULTISTAR0" value="" x="37.592" y="26.67" smashed="yes" rot="MR0"/>
 <element name="U$6" library="output" package="#PWR#0" value="" x="35.306" y="34.925" smashed="yes" rot="MR0"/>
 <element name="LOGO5" library="SparkFun-Aesthetics" package="SFE_LOGO_NAME_.2" value="SFE_LOGO_NAME.2_INCH" x="33.02" y="29.21" smashed="yes"/>
+<element name="U$1" library="output" package="OSHW_NOT_OSHA0" value="" x="38.989" y="19.05" smashed="yes" rot="MR0"/>
 </elements>
 <signals>
